Commit message: Added notebook notes fixes:  * Calculation inertia for base, wheels, caster  * Add weight to total 25, base 23 kilos, 2 wheels 1 kilo each.  * Fix naming on joints to be more descriptive  * Add gazebo tag for removing friction on casters

File: my_rb1_description/urdf/my_rb1_robot.urdf (robot description, URDF)
Before this commit: robot robot, 7 links, 6 joints
Links:
- link base_footprint: mass 21 -> None
- link base_link: mass 21 -> 23
- link front_laser: mass 21 -> None
Joints:
- removed joint joint_base_back_caster
- removed joint joint_base_base_footprint
- removed joint joint_base_front_caster
- removed joint joint_base_front_laser
- removed joint joint_base_left_wheel
- removed joint joint_base_right_wheel
- added joint joint_back_caster_to_base: type fixed, parent base_link, child back_caster, origin xyz=-0.1 0 -0.15 rpy=0 0 0
- added joint joint_base_to_base_footprint: type fixed, parent base_footprint, child base_link, origin xyz=0 0 0.15 rpy=0 0 0
- added joint joint_front_caster_to_base: type fixed, parent base_link, child front_caster, origin xyz=0.1 0 -0.15 rpy=0 0 0
- added joint joint_front_laser_to_base: type fixed, parent base_link, child front_laser, origin xyz=0.25 0 0.075 rpy=3.14159 0 0
- added joint joint_left_wheel_to_base: type continuous, parent base_link, child left_wheel, origin xyz=0 -0.2 -0.15 rpy=0 0 0, axis 0 1 0, limit effort=10000 velocity=1000
- added joint joint_right_wheel_to_base: type continuous, parent base_link, child right_wheel, origin xyz=0 0.2 -0.15 rpy=0 0 0, axis 0 1 0, limit effort=10000 velocity=1000

Commit message: Adding laser and diff driver plugins to model
Model Fixes:
 * Incresed wheels size
 * Switch wheels sides
 * Fix caster gazebo tag naming

File: my_rb1_description/urdf/my_rb1_robot.urdf (robot description, URDF)
Before this commit: robot robot, 7 links, 6 joints
Links:
- link left_wheel: geometry collision cylinder length=0.04 radius=0.025; visual cylinder length=0.04 radius=0.025
- link right_wheel: geometry collision cylinder length=0.04 radius=0.025; visual cylinder length=0.04 radius=0.025
Joints:
- joint joint_left_wheel_to_base: origin xyz=0 -0.2 -0.15 rpy=0 0 0 -> xyz=0 0.2 -0.15 rpy=0 0 0
- joint joint_right_wheel_to_base: origin xyz=0 0.2 -0.15 rpy=0 0 0 -> xyz=0 -0.2 -0.15 rpy=0 0 0
