Commit message: Adding xacro to my_rb1_robot model

File: my_rb1_description/urdf/my_rb1_robot.xacro (robot description, xacro)
@@ -1,4 +1,10 @@
 <?xml version="1.0" ?>
-<robot name="robot">
+<robot name="robot"  xmlns:xacro="http://www.ros.org/wiki/xacro">
+    <!-- Custom properties -->
+        <xacro:include filename="$(find my_rb1_description)/urdf/my_rb1_robot.gazebo" />
+        <xacro:property name="base_mass" value="23" />
+        <xacro:property name="default_mass" value="1" />
+        <xacro:property name="pi" value="3.1415926535897931" />
+        <xacro:property name="h_pi" value="${pi / 2}" />
     <!-- Base -->
         <!-- Base footprint -->
@@ -8,5 +14,5 @@
         <link name="base_link">
             <inertial>
-                <mass value="23" />
+                <mass value="${base_mass}" />
                 <origin xyz="0 0 0" rpy="0 0 0" />
                 <inertia ixx="0.5319" iyy="0.5319" izz="0.7188" ixy="0" ixz="0" iyz="0" />
@@ -33,10 +39,10 @@
         <link name="left_wheel">
             <inertial>
-                <mass value="1" />
+                <mass value="${default_mass}" />
                 <origin xyz="0 0 0" rpy="0 0 0" />
                 <inertia ixx="0.0001896" iyy="0.0001896" izz="0.0003125" ixy="0" ixz="0" iyz="0" />
             </inertial>
             <collision>
-                <origin rpy="1.57079633 0 0" xyz="0 0 0" />
+                <origin rpy="${h_pi} 0 0" xyz="0 0 0" />
                 <geometry>
                     <cylinder length="0.04" radius="0.025"/>
@@ -44,5 +50,5 @@
             </collision>
             <visual>
-                <origin rpy="1.57079633 0 0" xyz="0 0 0" />
+                <origin rpy="${h_pi} 0 0" xyz="0 0 0" />
                 <geometry>
                     <cylinder length="0.04" radius="0.025"/>
@@ -62,10 +68,10 @@
         <link name="right_wheel">
             <inertial>
-                <mass value="1" />
+                <mass value="${default_mass}" />
                 <origin xyz="0 0 0" rpy="0 0 0" />
                 <inertia ixx="0.0001896" iyy="0.0001896" izz="0.0003125" ixy="0" ixz="0" iyz="0" />
             </inertial>
             <collision>
-                <origin rpy="1.57079633 0 0" xyz="0 0 0" />
+                <origin rpy="${h_pi} 0 0" xyz="0 0 0" />
                 <geometry>
                     <cylinder length="0.04" radius="0.025"/>
@@ -73,5 +79,5 @@
             </collision>
             <visual>
-                <origin rpy="1.57079633 0 0" xyz="0 0 0" />
+                <origin rpy="${h_pi} 0 0" xyz="0 0 0" />
                 <geometry>
                     <cylinder length="0.04" radius="0.025"/>
@@ -92,5 +98,5 @@
         <link name="front_caster">
             <inertial>
-                <mass value="1" />
+                <mass value="${default_mass}" />
                 <origin xyz="0 0 0" rpy="0 0 0" />
                 <inertia ixx="0.00026667" ixy="0.00026667" izz="0.00026667" ixz="0" iyy="0.002526666666667" iyz="0" />
@@ -130,5 +136,5 @@
         <link name="back_caster">
             <inertial>
-                <mass value="1" />
+                <mass value="${default_mass}" />
                 <origin xyz="0 0 0" rpy="0 0 0" />
                 <inertia ixx="0.00026667" ixy="0.00026667" izz="0.00026667" ixz="0" iyy="0.002526666666667" iyz="0" />
@@ -171,65 +177,7 @@
         <!-- Joint - front laser - base -->
         <joint name="joint_front_laser_to_base" type="fixed">
-            <origin rpy="3.14159 0 0" xyz="0.25 0 0.075" />
+            <origin rpy="${pi} 0 0" xyz="0.25 0 0.075" />
             <child link="front_laser" />
             <parent link="base_link" />
         </joint>
-    <!-- Gazebo tags -->
-        <gazebo reference="front_caster">
-            <mu1>0</mu1>
-            <mu2>0</mu2>
-        </gazebo>
-        <gazebo reference="back_caster">
-            <mu1>0</mu1>
-            <mu2>0</mu2>
-        </gazebo>
-        <gazebo reference="base_link">
-            <material>Gazebo/Black</material>
-        </gazebo>
-        <gazebo>
-            <plugin filename="libgazebo_ros_diff_drive.so" name="differential_drive_controller">
-                <alwaysOn>true</alwaysOn>
-                <updateRate>20</updateRate>
-                <leftJoint>joint_left_wheel_to_base</leftJoint>
-                <rightJoint>joint_right_wheel_to_base</rightJoint>
-                <wheelSeparation>0.4</wheelSeparation>
-                <wheelDiameter>0.05</wheelDiameter>
-                <torque>10</torque>
-                <commandTopic>cmd_vel</commandTopic>
-                <odometryTopic>odom</odometryTopic>
-                <odometryFrame>odom</odometryFrame>
-                <robotBaseFrame>base_link</robotBaseFrame>
-            </plugin>
-        </gazebo>
-        <gazebo reference="front_laser">
-            <sensor type="ray" name="head_hokuyo_sensor">
-                <pose>0 0 0 0 0 0</pose>
-                <visualize>true</visualize>
-                <update_rate>20</update_rate>
-                <ray>
-                    <scan>
-                        <horizontal>
-                            <samples>720</samples>
-                            <resolution>1</resolution>
-                            <min_angle>-1.570796</min_angle>
-                            <max_angle>1.570796</max_angle>
-                        </horizontal>
-                    </scan>
-                    <range>
-                        <min>0.20</min>
-                        <max>10.0</max>
-                        <resolution>0.01</resolution>
-                    </range>
-                    <noise>
-                        <type>gaussian</type>
-                        <mean>0.0</mean>
-                        <stddev>0.01</stddev>
-                    </noise>
-                </ray>
-                <plugin name="gazebo_ros_head_hokuyo_controller" filename="libgazebo_ros_laser.so">
-                    <topicName>/scan</topicName>
-                    <frameName>sensor_laser</frameName>
-                </plugin>
-            </sensor>
-        </gazebo>
 </robot>
